File: manhattan.sch (KiCad schematic (older format))
At the start: 13 parts

Commit message: Microcontroller and USB mostly hooked up
Parts:
- added C? (x6): 220n, symbol C
- added C? (x11): 100n, symbol C
- added C? (x3): 100u, symbol CP1
- added C? (x2): 22pF, symbol C
- added C?: 1uF, symbol C
- added E0-CONN, Y-CONN, Z-CONN: CONN_4, symbol CONN_4
- added J?: USB, symbol USB
- added R? (x6): 0.05R, symbol R
- added R? (x4): 100K, symbol R
- added R? (x3): 0R, symbol R
- added R? (x2): 22, symbol R
- added SW?: SW_PUSH, symbol SW_PUSH
- added X?: CRYSTAL, symbol CRYSTAL
- added Y-DRIVER, Z-DRIVER, Z-DRIVER?: A4982, symbol A4982
- gave numbers to parts that had none: 2
Connections:
- net AGND: now also R?.2, R?.2, R?.2, R?.2, R?.2, R?.2
- net MOTGND: now also X-DRIVER.13 (GND1), X-DRIVER.24 (GND2), C?.1, C?.1, C?.1, C?.1, C?.1, C?.1, C?.2, C?.2, C?.2, C?.2, C?.2, C?.2, R?.1, R?.1, R?.1, Y-DRIVER.13 (GND1), Y-DRIVER.24 (GND2), Y-DRIVER.EPAD (PAD), Z-DRIVER.13 (GND1), Z-DRIVER.24 (GND2), Z-DRIVER.EPAD (PAD), Z-DRIVER?.13 (GND1), Z-DRIVER?.24 (GND2), Z-DRIVER?.EPAD (PAD)
- net VCC: now also U?.21 (VCC), U?.52 (VCC), U?.64 (AVCC), C?.2, C?.2, C?.2, R?.1, R?.1, R?.1, R?.1, Y-DRIVER.10 (VDD), Z-DRIVER.10 (VDD), Z-DRIVER?.10 (VDD)
- net VMOT: now also C?.1, C?.1, C?.1, C?.1, C?.1, C?.1, C?.2, C?.2, C?.2, Y-DRIVER.16 (VBB1), Y-DRIVER.21 (VBB2), Z-DRIVER.16 (VBB1), Z-DRIVER.21 (VBB2), Z-DRIVER?.16 (VBB1), Z-DRIVER?.21 (VBB2)
- net at U?.20 (RESET\): now also R?.2, SW?.2
- net LOGICGND: now reaches U?.22 (GND)
- net LOGICGND: now also U?.53 (GND), U?.6 (UGnd), U?.63 (AGND), C?.2, C?.2, C?.2, C?.2, C?.2, J?.4 (GND), SW?.1
- net at U?.23 (XTAL2): now also C?.1, X?.2
- net at U?.24 (XTAL1): now also C?.1, X?.1
- net at U?.3 (UVcc): now also U?.8 (VBus), C?.1, J?.1 (Vbus)
- net at U?.4 (D-): now also R?.1
- net at U?.5 (D+): now also R?.1
- net at U?.62 (AREF): now also C?.1
- net at U?.7 (UCap): now also C?.1
- net X-STEP: now reaches X-DRIVER.11 (STEP)
- net X-DIR: now reaches X-DRIVER.14 (DIR)
- net X-EN: now reaches X-DRIVER.23 (ENABLE)
- net X-MS1: now reaches X-DRIVER.5 (MS1)
- net X-MS2: now reaches X-DRIVER.6 (MS2)
- net XREF renamed X-REF
- new net: R?.1, Y-DRIVER.17 (SENSE1)
- new net: R?.1, Y-DRIVER.20 (SENSE2)
- new net: Y-CONN.1 (P1), Y-DRIVER.22 (OUT2B)
- new net: Y-CONN.2 (P2), Y-DRIVER.19 (OUT2A)
- new net: Y-CONN.3 (P3), Y-DRIVER.15 (OUT1B)
- new net: Y-CONN.4 (P4), Y-DRIVER.18 (OUT1A)
- new net: R?.2, Y-DRIVER.7 (RESET), Y-DRIVER.9 (SLEEP)
- new net: R?.2, Y-DRIVER.8 (ROSC)
- new net: C?.2, Y-DRIVER.4 (VREG)
- new net: C?.1, Y-DRIVER.3 (VCP)
- new net: C?.1, Y-DRIVER.2 (CP2)
- new net: C?.2, Y-DRIVER.1 (CP1)
- new net: C?.2, Z-DRIVER.1 (CP1)
- new net: Z-CONN.3 (P3), Z-DRIVER.15 (OUT1B)
- new net: R?.1, Z-DRIVER.17 (SENSE1)
- new net: Z-CONN.4 (P4), Z-DRIVER.18 (OUT1A)
- new net: Z-CONN.2 (P2), Z-DRIVER.19 (OUT2A)
- new net: C?.1, Z-DRIVER.2 (CP2)
- new net: R?.1, Z-DRIVER.20 (SENSE2)
- new net: Z-CONN.1 (P1), Z-DRIVER.22 (OUT2B)
- new net: C?.1, Z-DRIVER.3 (VCP)
- new net: C?.2, Z-DRIVER.4 (VREG)
- new net: R?.2, Z-DRIVER.7 (RESET), Z-DRIVER.9 (SLEEP)
- new net: R?.2, Z-DRIVER.8 (ROSC)
- new net: R?.1, Z-DRIVER?.17 (SENSE1)
- new net: R?.1, Z-DRIVER?.20 (SENSE2)
- new net: E0-CONN.1 (P1), Z-DRIVER?.22 (OUT2B)
- new net: E0-CONN.2 (P2), Z-DRIVER?.19 (OUT2A)
- new net: E0-CONN.3 (P3), Z-DRIVER?.15 (OUT1B)
- new net: E0-CONN.4 (P4), Z-DRIVER?.18 (OUT1A)
- new net: R?.2, Z-DRIVER?.7 (RESET), Z-DRIVER?.9 (SLEEP)
- new net: R?.2, Z-DRIVER?.8 (ROSC)
- new net: C?.2, Z-DRIVER?.4 (VREG)
- new net: C?.1, Z-DRIVER?.3 (VCP)
- new net: C?.1, Z-DRIVER?.2 (CP2)
- new net: C?.2, Z-DRIVER?.1 (CP1)
- new net: J?.2 (D-), R?.2
- new net: J?.3 (D+), R?.2
- new net E0-DIR: Z-DRIVER?.14 (DIR)
- new net E0-EN: Z-DRIVER?.23 (ENABLE)
- new net E0-MS1: Z-DRIVER?.5 (MS1)
- new net E0-MS2: Z-DRIVER?.6 (MS2)
- new net E0-REF: Z-DRIVER?.12 (REF)
- new net E0-STEP: Z-DRIVER?.11 (STEP)
- new net Y-DIR: Y-DRIVER.14 (DIR)
- new net Y-EN: Y-DRIVER.23 (ENABLE)
- new net Y-MS1: Y-DRIVER.5 (MS1)
- new net Y-MS2: Y-DRIVER.6 (MS2)
- new net Y-REF: Y-DRIVER.12 (REF)
- new net Y-STEP: Y-DRIVER.11 (STEP)
- new net Z-DIR: Z-DRIVER.14 (DIR)
- new net Z-EN: Z-DRIVER.23 (ENABLE)
- new net Z-MS1: Z-DRIVER.5 (MS1)
- new net Z-MS2: Z-DRIVER.6 (MS2)
- new net Z-REF: Z-DRIVER.12 (REF)
- new net Z-STEP: Z-DRIVER.11 (STEP)
- no-connect marks 0 -> 2
Other:
- note added: "E0 axis stepper module"
- note added: "Y axis stepper module"
- note added: "Z axis stepper module"
- moved on the sheet: C?, R?, X-CONN, X-DRIVER

Commit message: Schematic more or less done
TODO:
- FTDI headers
- Expansion I/O headers
Parts:
- added BED_CONN, FAN_CONN, HOTEND_CONN, P? (x3): CONN_2, symbol CONN_2
- added C? (x3): 100n, symbol C
- added C? (x2): 10uF, symbol C
- added C?: 220uF, symbol CP1
- added C? (x3): 10uF, symbol CP1
- added D?: LED, symbol LED
- added ISP: CONN_3X2, symbol CONN_3X2
- added J?: MICROSD-JT10, symbol MICROSD-JT10
- added JP?, USBPWR: JUMPER, symbol JUMPER
- added K? (x4): CONN_3, symbol CONN_3
- added P?: CONN_6, symbol CONN_6
- added Q? (x3): MOSFET_N, symbol MOSFET_N
- added R? (x4): 100K, symbol R
- added R? (x2): 4K7 1%, symbol R
- added R?: R, symbol R
- added R? (x3): 100, symbol R
- added U?: MC78M05CDTX, symbol MC78M05CDTX
- added U?: AP7313, symbol AP7313
- added U?: TXB0104, symbol TXB0104
- X?: value CRYSTAL -> 16.000
- gave numbers to parts that had none: 2
Connections:
- net labels added: +3.3V, B-THERM, BED, E-STOP, E-THERM, FAN, HOTEND, MISO, MOSI, RESET, SCLK, SDCLK, SDCS, SDCSH, SDDET, SDDI, SDDO, X-STOP, Y-STOP, Z-STOP
- wire segments 277 -> 423
- no-connect marks 2 -> 4
Other:
- note added: "Endstops"
- note added: "ISP"
- note added: "MOSFETs"
- note added: "Microcontroller and USB"
- note added: "Power"
- note added: "Thermistors"
- note added: "microSD"
- moved on the sheet: C?, J?, MCU, R?, RESETSW, X?

Commit message: FTDI and expansion header done
Parts:
- added P?: CONN_7X2, symbol CONN_7X2
Connections:
- net labels added: RX, TX
- wire segments 423 -> 439
Other:
- note added: "Expansion header"
- note added: "FTDI"
- moved on the sheet: P?
Changed lines of the file:
@@
-EESchema Schematic File Version 2  date Sat 10 Mar 2012 03:10:11 PM EST
+EESchema Schematic File Version 2  date Sat 10 Mar 2012 04:14:28 PM EST
 LIBS:manhattan
 LIBS:power
@@
 Comment4 ""
 $EndDescr
-Wire Wire Line
-	9900 6150 9900 6450
-Wire Wire Line
-	9900 6450 9800 6450
-Wire Wire Line
-	10050 6350 9800 6350
-Wire Wire Line
-	10050 6550 9800 6550
-Wire Wire Line
-	9900 6750 9800 6750
+Text Notes 10150 6100 0    120  ~ 0
+Expansion header
+Wire Notes Line
+	12450 5950 10150 5950
+Wire Notes Line
+	12450 5950 12450 7300
+Wire Notes Line
+	12450 7300 10150 7300
+Wire Notes Line
+	10150 7300 10150 5950
+Wire Wire Line
+	12200 6900 11750 6900
+Wire Wire Line
+	12200 6700 11750 6700
+Wire Wire Line
+	12200 6500 11750 6500
+Wire Wire Line
+	10500 7000 10950 7000
+Wire Wire Line
+	10500 6800 10950 6800
+Wire Wire Line
+	10500 6600 10950 6600
+Wire Wire Line
+	10500 6400 10950 6400
+Wire Wire Line
+	5400 9800 5150 9800
+Wire Wire Line
+	9750 6600 9500 6600
+Wire Wire Line
+	9750 6500 9500 6500
+Wire Wire Line
+	9600 6900 9500 6900
 Connection ~ 15050 5750
 Wire Wire Line
@@
 	16450 4100 12550 4100
 Wire Wire Line
-	9800 6650 9900 6650
-Wire Wire Line
-	9900 6650 9900 6900
-Connection ~ 9900 6750
-Wire Wire Line
-	10050 6250 9800 6250
+	9500 6800 9600 6800
+Wire Wire Line
+	9600 6800 9600 7050
+Connection ~ 9600 6900
+Wire Wire Line
+	9750 6400 9500 6400
+Wire Wire Line
+	9500 6700 9850 6700
+Wire Wire Line
+	9850 6700 9850 6300
+Wire Wire Line
+	5400 9700 5150 9700
+Wire Notes Line
+	8550 7300 8550 5950
+Wire Notes Line
+	8550 7300 10100 7300
+Wire Notes Line
+	10100 7300 10100 5950
+Wire Notes Line
+	10100 5950 8550 5950
+Wire Wire Line
+	10500 6500 10950 6500
+Wire Wire Line
+	10500 6700 10950 6700
+Wire Wire Line
+	10500 6900 10950 6900
+Wire Wire Line
+	12200 6400 11750 6400
+Wire Wire Line
+	12200 6600 11750 6600
+Wire Wire Line
+	12200 6800 11750 6800
+Wire Wire Line
+	12200 7000 11750 7000
+$Comp
+L CONN_7X2 P?
+U 1 1 4F5BC3D9
+P 11350 6700
+F 0 "P?" H 11350 7100 60  0000 C CNN
+F 1 "CONN_7X2" V 11350 6700 60  0000 C CNN
+	1    11350 6700
+	1    0    0    -1
+$EndComp
+Text Notes 8550 6100 0    120  ~ 0
+FTDI
+Text Label 5150 9800 0    60   ~ 0
+RX
+Text Label 5150 9700 0    60   ~ 0
+TX
+Text Label 9500 6600 0    60   ~ 0
+RX
+Text Label 9500 6400 0    60   ~ 0
+RESET
+Text Label 9500 6500 0    60   ~ 0
+TX
 $Comp
 L VCC #PWR?
 U 1 1 4F5BB50E
-P 9900 6150
-F 0 "#PWR?" H 9900 6300 30  0001 C CNN
-F 1 "VCC" H 9900 6300 30  0000 C CNN
-	1    9900 6150
+P 9850 6300
+F 0 "#PWR?" H 9850 6450 30  0001 C CNN
+F 1 "VCC" H 9850 6450 30  0000 C CNN
+	1    9850 6300
 	1    0    0    -1
 $EndComp
@@
 L LOGICGND #PWR?
 U 1 1 4F5BB4F6
-P 9900 6950
-F 0 "#PWR?" H 9900 6950 30  0001 C CNN
-F 1 "LOGICGND" H 9900 6880 30  0001 C CNN
-	1    9900 6950
+P 9600 7100
+F 0 "#PWR?" H 9600 7100 30  0001 C CNN
+F 1 "LOGICGND" H 9600 7030 30  0001 C CNN
+	1    9600 7100
 	1    0    0    -1
 $EndComp
@@
 L CONN_6 P?
 U 1 1 4F5BB4F1
-P 9450 6500
-F 0 "P?" V 9400 6500 60  0000 C CNN
-F 1 "CONN_6" V 9500 6500 60  0000 C CNN
-	1    9450 6500
+P 9150 6650
+F 0 "P?" V 9100 6650 60  0000 C CNN
+F 1 "CONN_6" V 9200 6650 60  0000 C CNN
+	1    9150 6650
 	-1   0    0    1
 $EndComp

Commit message: Digipot for current control
Parts:
- added DP?: MCP4362, symbol MCP4362
- added R? (x4): 20K, symbol R
Connections:
- net labels added: E-REF, POTCS, POTSCK, POTSDI, POTSDO
- wire segments 439 -> 467
- no-connect marks 4 -> 6
Other:
- note added: "Stepper current control"
Changed lines of the file:
@@
-EESchema Schematic File Version 2  date Sat 10 Mar 2012 04:14:28 PM EST
+EESchema Schematic File Version 2  date Mon 12 Mar 2012 12:50:54 PM EDT
 LIBS:manhattan
 LIBS:power
@@
 Sheet 1 1
 Title ""
-Date "10 mar 2012"
+Date "12 mar 2012"
 Rev ""
 Comp ""
@@
 Comment4 ""
 $EndDescr
-Text Notes 10150 6100 0    120  ~ 0
-Expansion header
+Text Notes 8550 7500 0    120  ~ 0
+Stepper current control
+Wire Notes Line
+	12450 7350 8550 7350
+Wire Notes Line
+	12450 7350 12450 9100
+Wire Notes Line
+	12450 9100 8550 9100
+Wire Notes Line
+	8550 9100 8550 7350
+Connection ~ 11900 8050
+Wire Wire Line
+	11150 8050 11900 8050
+Wire Wire Line
+	9750 8250 10050 8250
+Wire Wire Line
+	9750 8050 10050 8050
+Wire Wire Line
+	9750 8550 10050 8550
+Wire Wire Line
+	11450 7850 11150 7850
+Connection ~ 11200 8450
+Wire Wire Line
+	11200 7950 11200 8900
+Wire Wire Line
+	11200 7950 11150 7950
+Connection ~ 10600 8900
+Wire Wire Line
+	11200 8900 10000 8900
+Connection ~ 11900 7750
+Wire Wire Line
+	11900 7650 11900 8650
+Wire Wire Line
+	11900 8650 11700 8650
+Connection ~ 9300 7750
+Wire Wire Line
+	9300 7650 9300 8650
+Wire Wire Line
+	9300 8650 9500 8650
+Wire Wire Line
+	10000 8650 10050 8650
+Wire Wire Line
+	11150 7750 11200 7750
+Wire Wire Line
+	10000 7750 10050 7750
+Wire Wire Line
+	11150 8650 11200 8650
+Wire Wire Line
+	9300 7750 9500 7750
+Wire Wire Line
+	11900 7750 11700 7750
+Wire Wire Line
+	10000 8450 10050 8450
+Wire Wire Line
+	10600 8900 10600 9000
+Wire Wire Line
+	10050 7950 10000 7950
+Wire Wire Line
+	10000 7950 10000 8900
+Connection ~ 10000 8450
+Wire Wire Line
+	11450 8550 11150 8550
+Wire Wire Line
+	9750 7850 10050 7850
 Wire Notes Line
 	12450 5950 10150 5950
@@
 Wire Wire Line
 	12200 7000 11750 7000
+Wire Wire Line
+	11150 8450 11200 8450
+Wire Wire Line
+	9750 8150 10050 8150
+Wire Wire Line
+	10000 8350 10050 8350
+Connection ~ 10000 8350
+Wire Wire Line
+	11450 8150 11150 8150
+Connection ~ 11900 8350
+Connection ~ 11900 8250
+NoConn ~ 11150 8350
+NoConn ~ 11150 8250
+Text Label 11150 8150 0    60   ~ 0
+POTSDO
+$Comp
+L MCP4362 DP?
+U 1 1 4F5E2698
+P 10600 8200
+F 0 "DP?" H 10600 8750 60  0000 C CNN
+F 1 "MCP4362" H 10600 7650 60  0000 C CNN
+	1    10600 8200
+	1    0    0    -1
+$EndComp
+Text Label 9750 8250 0    60   ~ 0
+POTSDI
+Text Label 9750 8150 0    60   ~ 0
+POTSCK
+Text Label 9750 8050 0    60   ~ 0
+POTCS
+Text Label 9750 7950 0    60   ~ 0
+E-REF
+Text Label 11200 7950 0    60   ~ 0
+Z-REF
+Text Label 9750 8550 0    60   ~ 0
+Y-REF
+Text Label 11200 8550 0    60   ~ 0
+X-REF
+$Comp
+L LOGICGND #PWR?
+U 1 1 4F5E241E
+P 10600 9050
+F 0 "#PWR?" H 10600 9050 30  0001 C CNN
+F 1 "LOGICGND" H 10600 8980 30  0001 C CNN
+	1    10600 9050
+	1    0    0    -1
+$EndComp
+$Comp
+L VCC #PWR?
+U 1 1 4F5E2407
+P 11900 7650
+F 0 "#PWR?" H 11900 7800 30  0001 C CNN
+F 1 "VCC" H 11900 7800 30  0000 C CNN
+	1    11900 7650
+	1    0    0    -1
+$EndComp
+$Comp
+L VCC #PWR?
+U 1 1 4F5E2404
+P 9300 7650
+F 0 "#PWR?" H 9300 7800 30  0001 C CNN
+F 1 "VCC" H 9300 7800 30  0000 C CNN
+	1    9300 7650
+	1    0    0    -1
+$EndComp
+$Comp
+L R R?
+U 1 1 4F5E23E1
+P 11450 8650
+F 0 "R?" V 11530 8650 50  0000 C CNN
+F 1 "20K" V 11450 8650 50  0000 C CNN
+	1    11450 8650
+	0    1    1    0
+$EndComp
+$Comp
+L R R?
+U 1 1 4F5E23DC
+P 9750 8650
+F 0 "R?" V 9830 8650 50  0000 C CNN
+F 1 "20K" V 9750 8650 50  0000 C CNN
+	1    9750 8650
+	0    1    1    0
+$EndComp
+$Comp
+L R R?
+U 1 1 4F5E23D9
+P 11450 7750
+F 0 "R?" V 11530 7750 50  0000 C CNN
+F 1 "20K" V 11450 7750 50  0000 C CNN
+	1    11450 7750
+	0    1    1    0
+$EndComp
+$Comp
+L R R?
+U 1 1 4F5E23D6
+P 9750 7750
+F 0 "R?" V 9830 7750 50  0000 C CNN
+F 1 "20K" V 9750 7750 50  0000 C CNN
+	1    9750 7750
+	0    1    1    0
+$EndComp
+Text Notes 10150 6100 0    120  ~ 0
+Expansion header
 $Comp
 L CONN_7X2 P?

Commit message: Fuses
Parts:
- added F?: 20A, symbol FUSE
- added F?: 5A, symbol FUSE
Connections:
- wire segments 467 -> 470
Other:
- moved on the sheet: P?
Changed lines of the file:
@@
-EESchema Schematic File Version 2  date Mon 12 Mar 2012 12:50:54 PM EDT
+EESchema Schematic File Version 2  date Mon 12 Mar 2012 03:13:13 PM EDT
 LIBS:manhattan
 LIBS:power
@@
 Comment4 ""
 $EndDescr
-Text Notes 8550 7500 0    120  ~ 0
-Stepper current control
+Wire Wire Line
+	7800 7450 7800 7400
+Connection ~ 14250 4350
+Wire Wire Line
+	14250 4550 14250 4350
+Wire Wire Line
+	13450 4350 15950 4350
+Wire Wire Line
+	14800 5750 14800 5300
+Connection ~ 14800 5750
 Wire Notes Line
 	12450 7350 8550 7350
@@
 	15950 5750 12700 5750
 Connection ~ 14300 5750
-Wire Wire Line
-	14800 5750 14800 5300
 Connection ~ 13600 5750
 Wire Wire Line
@@
 	13600 4750 13600 4900
 Connection ~ 13450 4350
-Wire Wire Line
-	14800 4350 14800 4550
 Wire Notes Line
 	12450 4100 8550 4100
@@
 	6150 10300 6150 5950
 Wire Wire Line
-	7600 6400 7600 6550
-Wire Wire Line
-	7600 6550 7700 6550
+	7600 6200 7600 6350
+Wire Wire Line
+	7600 6350 7700 6350
 Connection ~ 7700 8000
 Wire Wire Line
@@
 	6150 5950 8450 5950
 Wire Wire Line
-	7700 6750 7600 6750
-Wire Wire Line
-	7600 6750 7600 6900
+	7700 6550 7600 6550
+Wire Wire Line
+	7600 6550 7600 6700
 Wire Wire Line
 	6800 8100 6800 7800
@@
 	13450 4550 13600 4550
 Wire Wire Line
-	13450 4350 15950 4350
-Wire Wire Line
 	15950 4350 15950 4550
-Connection ~ 14800 4350
 Wire Wire Line
 	14800 4750 14800 4900
@@
 Wire Wire Line
 	15050 5750 15050 5600
-Connection ~ 14800 5750
 Wire Notes Line
 	12550 5900 12550 4100
@@
 Connection ~ 11900 8350
 Connection ~ 11900 8250
+Wire Wire Line
+	14750 4550 14800 4550
+Wire Wire Line
+	7800 6900 7800 6850
+$Comp
+L MOTGND #PWR?
+U 1 1 4F5E4AAC
+P 7800 7500
+F 0 "#PWR?" H 7800 7500 30  0001 C CNN
+F 1 "MOTGND" H 7800 7430 30  0001 C CNN
+	1    7800 7500
+	1    0    0    -1
+$EndComp
+$Comp
+L FUSE F?
+U 1 1 4F5E4AA4
+P 7800 7150
+F 0 "F?" H 7900 7200 40  0000 C CNN
+F 1 "5A" H 7700 7100 40  0000 C CNN
+	1    7800 7150
+	0    1    1    0
+$EndComp
+$Comp
+L VMOT #PWR?
+U 1 1 4F5E4AA0
+P 7800 6850
+F 0 "#PWR?" H 7800 7000 30  0001 C CNN
+F 1 "VMOT" H 7800 7000 30  0000 C CNN
+	1    7800 6850
+	1    0    0    -1
+$EndComp
+$Comp
+L FUSE F?
+U 1 1 4F5E4A7C
+P 14500 4550
+F 0 "F?" H 14600 4600 40  0000 C CNN
+F 1 "20A" H 14400 4500 40  0000 C CNN
+	1    14500 4550
+	1    0    0    -1
+$EndComp
+Text Notes 8550 7500 0    120  ~ 0
+Stepper current control
 NoConn ~ 11150 8350
 NoConn ~ 11150 8250
@@
 L LOGICGND #PWR?
 U 1 1 4F5B9D07
-P 7600 6950
-F 0 "#PWR?" H 7600 6950 30  0001 C CNN
-F 1 "LOGICGND" H 7600 6880 30  0001 C CNN
-	1    7600 6950
+P 7600 6750
+F 0 "#PWR?" H 7600 6750 30  0001 C CNN
+F 1 "LOGICGND" H 7600 6680 30  0001 C CNN
+	1    7600 6750
 	1    0    0    -1
 $EndComp
@@
 L VMOT #PWR?
 U 1 1 4F5B9D04
-P 7600 6400
-F 0 "#PWR?" H 7600 6550 30  0001 C CNN
-F 1 "VMOT" H 7600 6550 30  0000 C CNN
-	1    7600 6400
+P 7600 6200
+F 0 "#PWR?" H 7600 6350 30  0001 C CNN
+F 1 "VMOT" H 7600 6350 30  0000 C CNN
+	1    7600 6200
 	1    0    0    -1
 $EndComp
@@
 L CONN_2 P?
 U 1 1 4F5B9CFE
-P 8050 6650
-F 0 "P?" V 8000 6650 40  0000 C CNN
-F 1 "CONN_2" V 8100 6650 40  0000 C CNN
-	1    8050 6650
-	1    0    0    -1
-$EndComp
+P 8050 6450
+F 0 "P?" V 8000 6450 40  0000 C CNN
+F 1 "CONN_2" V 8100 6450 40  0000 C CNN
+	1    8050 6450
+	1    0    0    -1
+$EndComp

Commit message: Stepper current control done
Parts:
- removed DP?: MCP4362, symbol MCP4362
- removed R? (x4): 20K, symbol R
- added C? (x2): 100n, symbol C
- added DP?: MCP4451, symbol MCP4451
- added R? (x4): 20K, symbol R
- F?: value 5A -> FUSE
Connections:
- net labels added: +12V, SCL, SDA
- net labels removed: POTCS, POTSCK, POTSDI, POTSDO
- wire segments 470 -> 465
- no-connect marks 6 -> 8
Other:
- moved on the sheet: F?

Commit message: Annotation
Parts:
- gave numbers to parts that had none: 97
- renumbered BED_CONN to BED_CONN1, E0-CONN to E0-CONN1, FAN_CONN to FAN_CONN1, HOTEND_CONN to HOTEND_CONN1, ISP to ISP1, MCU to MCU1, RESETSW to RESETSW1, USBPWR to USBPWR1, X-CONN to X-CONN1, X-DRIVER to X-DRIVER1, Y-CONN to Y-CONN1, Y-DRIVER to Y-DRIVER1, Z-CONN to Z-CONN1, Z-DRIVER to Z-DRIVER1
